File: Input.sch (KiCad schematic (older format))
At the start: 30 parts

Commit message: first layout
Parts:
- C18, C19, C20, C21, C22: renamed from C?; footprint (none) -> Capacitor_SMD:C_0603_1608Metric
- J4: renamed from J?; footprint (none) -> stmbl:RJ45_LED
- L2: renamed from L?; footprint (none) -> Inductor_SMD:L_0603_1608Metric
- R37, R38, R39, R40, R41, R42, R43, R44, R45, R46, R47, R48, R49, R50, R51, R52, R53, R54, R55: renamed from R?; footprint (none) -> Resistor_SMD:R_0603_1608Metric
- gave numbers to parts that had none: 4
