File: RS485Tranceiver.sch (KiCad schematic (older format))
At the start: 19 parts, among them J10 Conn_01x02, U13 SN75176AD

Commit message: updated RS422
Connections:
- net OUT renamed DATA
Changed lines of the file:
@@
 AR Path="/6072829D/60795F15/6072BD6B" Ref="#PWR0116"  Part="1"
 AR Path="/6072829D/60797D2F/6072BD6B" Ref="#PWR0122"  Part="1"
-F 0 "#PWR0130" H 8600 2950 50  0001 C CNN
+F 0 "#PWR0110" H 8600 2950 50  0001 C CNN
 F 1 "GND" H 8605 3027 50  0000 C CNN
 F 2 "" H 8600 3200 50  0001 C CNN
@@
 AR Path="/6072829D/60795F15/6073EDE6" Ref="#PWR0113"  Part="1"
 AR Path="/6072829D/60797D2F/6073EDE6" Ref="#PWR0119"  Part="1"
-F 0 "#PWR0125" H 3600 2550 50  0001 C CNN
+F 0 "#PWR0107" H 3600 2550 50  0001 C CNN
 F 1 "GND" H 3605 2627 50  0000 C CNN
 F 2 "" H 3600 2800 50  0001 C CNN
@@
 AR Path="/6072829D/60795F15/6073EDED" Ref="#PWR0111"  Part="1"
 AR Path="/6072829D/60797D2F/6073EDED" Ref="#PWR0117"  Part="1"
-F 0 "#PWR0123" H 3100 2550 50  0001 C CNN
+F 0 "#PWR0104" H 3100 2550 50  0001 C CNN
 F 1 "GND" H 3105 2627 50  0000 C CNN
 F 2 "" H 3100 2800 50  0001 C CNN
@@
 AR Path="/6072829D/60795F15/6073EE1A" Ref="#PWR0114"  Part="1"
 AR Path="/6072829D/60797D2F/6073EE1A" Ref="#PWR0120"  Part="1"
-F 0 "#PWR0126" H 3600 4050 50  0001 C CNN
+F 0 "#PWR0108" H 3600 4050 50  0001 C CNN
 F 1 "GND" H 3605 4127 50  0000 C CNN
 F 2 "" H 3600 4300 50  0001 C CNN
@@
 AR Path="/6072829D/60795F15/6073EE21" Ref="#PWR0112"  Part="1"
 AR Path="/6072829D/60797D2F/6073EE21" Ref="#PWR0118"  Part="1"
-F 0 "#PWR0124" H 3100 4050 50  0001 C CNN
+F 0 "#PWR0105" H 3100 4050 50  0001 C CNN
 F 1 "GND" H 3105 4127 50  0000 C CNN
 F 2 "" H 3100 4300 50  0001 C CNN
@@
 AR Path="/6072829D/60795F15/6073EE2E" Ref="#PWR0115"  Part="1"
 AR Path="/6072829D/60797D2F/6073EE2E" Ref="#PWR0121"  Part="1"
-F 0 "#PWR0129" H 6350 2450 50  0001 C CNN
+F 0 "#PWR0109" H 6350 2450 50  0001 C CNN
 F 1 "GND" H 6355 2527 50  0000 C CNN
 F 2 "" H 6350 2700 50  0001 C CNN
@@
 Text HLabel 10200 1950 2    50   Input ~ 0
 VCC
-Text HLabel 9200 2200 2    50   Input ~ 0
-OUT
+Text HLabel 9200 2200 2    50   BiDi ~ 0
+DATA
 $EndSCHEMATC
