File: HF_Ctrl.sch (KiCad schematic (older format))
At the start: 15 parts

Commit message: first layout
Parts:
- D7: renamed from D?; footprint (none) -> Diode_SMD:D_0603_1608Metric
- J7: renamed from J?; footprint (none) -> Connector_Dsub:DSUB-9_Female_Vertical_P2.77x2.84mm
- J8: renamed from J?; footprint (none) -> stmbl:RM3.5_1x2
- K1: renamed from K?; footprint (none) -> Relay_THT:Relay_DPDT_Omron_G6S-2
- R55, R57, R59, R60: renamed from R?; footprint (none) -> Resistor_SMD:R_0603_1608Metric
- R56, R58: renamed from R?; footprint (none) -> Resistor_SMD:R_1206_3216Metric_Pad1.30x1.75mm_HandSolder
- gave numbers to parts that had none: 5
Changed lines of the file:
@@
 $Descr A4 11693 8268
 encoding utf-8
-Sheet 9 9
+Sheet 12 17
 Title ""
 Date ""
@@
 P 7150 800
 AR Path="/60660B68/607E635B" Ref="#PWR?"  Part="1"
-AR Path="/607E0323/607E635B" Ref="#PWR?"  Part="1"
-F 0 "#PWR?" H 7150 650 50  0001 C CNN
+AR Path="/607E0323/607E635B" Ref="#PWR097"  Part="1"
+F 0 "#PWR097" H 7150 650 50  0001 C CNN
 F 1 "+24V" H 7165 973 50  0000 C CNN
 F 2 "" H 7150 800 50  0001 C CNN
@@
 	7250 1850 7350 1850
 $Comp
-L Transistor_FET:AO3400A Q?
+L Transistor_FET:AO3400A Q8
 U 1 1 607F6434
 P 5500 2400
-F 0 "Q?" H 5705 2446 50  0000 L CNN
+F 0 "Q8" H 5705 2446 50  0000 L CNN
 F 1 "AO3400A" H 5705 2355 50  0000 L CNN
 F 2 "Package_TO_SOT_SMD:SOT-23" H 5700 2325 50  0001 L CIN
@@
 	5600 1750 7350 1750
 $Comp
-L AR2ISS:R R?
+L AR2ISS:R R57
 U 1 1 607FEDFC
 P 5200 2600
-F 0 "R?" H 5270 2646 50  0000 L CNN
+F 0 "R57" H 5270 2646 50  0000 L CNN
 F 1 "100k" H 5270 2555 50  0000 L CNN
-F 2 "" V 5130 2600 50  0001 C CNN
+F 2 "Resistor_SMD:R_0603_1608Metric" V 5130 2600 50  0001 C CNN
 F 3 "~" H 5200 2600 50  0001 C CNN
 	1    5200 2600
@@
 	3950 2450 3950 2400
 $Comp
-L AR2ISS:R R?
+L AR2ISS:R R55
 U 1 1 607FE5A7
 P 3950 2600
-F 0 "R?" H 4020 2646 50  0000 L CNN
+F 0 "R55" H 4020 2646 50  0000 L CNN
 F 1 "100k" H 4020 2555 50  0000 L CNN
-F 2 "" V 3880 2600 50  0001 C CNN
+F 2 "Resistor_SMD:R_0603_1608Metric" V 3880 2600 50  0001 C CNN
 F 3 "~" H 3950 2600 50  0001 C CNN
 	1    3950 2600
@@
 $EndComp
 $Comp
-L Transistor_FET:AO3400A Q?
+L Transistor_FET:AO3400A Q7
 U 1 1 607EDBCE
 P 4250 2400
-F 0 "Q?" H 4455 2446 50  0000 L CNN
+F 0 "Q7" H 4455 2446 50  0000 L CNN
 F 1 "AO3400A" H 4450 2300 50  0000 L CNN
 F 2 "Package_TO_SOT_SMD:SOT-23" H 4450 2325 50  0001 L CIN
@@
 Connection ~ 5200 2400
 $Comp
-L Connector_Generic:Conn_01x02 J?
+L Connector_Generic:Conn_01x02 J8
 U 1 1 6081272B
 P 9250 4900
-F 0 "J?" H 9330 4892 50  0000 L CNN
+F 0 "J8" H 9330 4892 50  0000 L CNN
 F 1 "Conn_01x02" H 9330 4801 50  0000 L CNN
-F 2 "" H 9250 4900 50  0001 C CNN
+F 2 "stmbl:RM3.5_1x2" H 9250 4900 50  0001 C CNN
 F 3 "~" H 9250 4900 50  0001 C CNN
 	1    9250 4900
@@
 $EndComp
 $Comp
-L Transistor_FET:AO3400A Q?
+L Transistor_FET:AO3400A Q9
 U 1 1 608139C2
 P 6550 5100
-F 0 "Q?" H 6755 5146 50  0000 L CNN
+F 0 "Q9" H 6755 5146 50  0000 L CNN
 F 1 "AO3400A" H 6755 5055 50  0000 L CNN
 F 2 "Package_TO_SOT_SMD:SOT-23" H 6750 5025 50  0001 L CIN
@@
 $EndComp
 $Comp
-L AR2ISS:R R?
+L AR2ISS:R R59
 U 1 1 6081705A
 P 6200 5350
-F 0 "R?" H 6270 5396 50  0000 L CNN
+F 0 "R59" H 6270 5396 50  0000 L CNN
 F 1 "100k" H 6270 5305 50  0000 L CNN
-F 2 "" V 6130 5350 50  0001 C CNN
+F 2 "Resistor_SMD:R_0603_1608Metric" V 6130 5350 50  0001 C CNN
 F 3 "~" H 6200 5350 50  0001 C CNN
 	1    6200 5350
@@
 P 6650 5600
 AR Path="/60660B68/6081A518" Ref="#PWR?"  Part="1"
-AR Path="/607E0323/6081A518" Ref="#PWR?"  Part="1"
-F 0 "#PWR?" H 6650 5350 50  0001 C CNN
+AR Path="/607E0323/6081A518" Ref="#PWR095"  Part="1"
+F 0 "#PWR095" H 6650 5350 50  0001 C CNN
 F 1 "GND" H 6655 5427 50  0000 C CNN
 F 2 "" H 6650 5600 50  0001 C CNN
@@
 P 5600 2850
 AR Path="/60660B68/607FD23E" Ref="#PWR?"  Part="1"
-AR Path="/607E0323/607FD23E" Ref="#PWR?"  Part="1"
-F 0 "#PWR?" H 5600 2600 50  0001 C CNN
+AR Path="/607E0323/607FD23E" Ref="#PWR094"  Part="1"
+F 0 "#PWR094" H 5600 2600 50  0001 C CNN
 F 1 "GND" H 5605 2677 50  0000 C CNN
 F 2 "" H 5600 2850 50  0001 C CNN
@@
 P 4350 2850
 AR Path="/60660B68/607FD51C" Ref="#PWR?"  Part="1"
-AR Path="/607E0323/607FD51C" Ref="#PWR?"  Part="1"
-F 0 "#PWR?" H 4350 2600 50  0001 C CNN
+AR Path="/607E0323/607FD51C" Ref="#PWR093"  Part="1"
+F 0 "#PWR093" H 4350 2600 50  0001 C CNN
 F 1 "GND" H 4355 2677 50  0000 C CNN
 F 2 "" H 4350 2850 50  0001 C CNN
@@
 	3950 2750 3950 2800
 $Comp
-L AR2ISS:R R?
+L AR2ISS:R R56
 U 1 1 6082428F
 P 4350 2000
-F 0 "R?" H 4420 2046 50  0000 L CNN
+F 0 "R56" H 4420 2046 50  0000 L CNN
 F 1 "50" H 4420 1955 50  0000 L CNN
-F 2 "" V 4280 2000 50  0001 C CNN
+F 2 "Resistor_SMD:R_1206_3216Metric_Pad1.30x1.75mm_HandSolder" V 4280 2000 50  0001 C CNN
 F 3 "~" H 4350 2000 50  0001 C CNN
 	1    4350 2000
@@
 $EndComp
 $Comp
-L AR2ISS:R R?
+L AR2ISS:R R58
 U 1 1 60834F37
 P 5600 2000
-F 0 "R?" H 5670 2046 50  0000 L CNN
+F 0 "R58" H 5670 2046 50  0000 L CNN
 F 1 "50" H 5670 1955 50  0000 L CNN
-F 2 "" V 5530 2000 50  0001 C CNN
+F 2 "Resistor_SMD:R_1206_3216Metric_Pad1.30x1.75mm_HandSolder" V 5530 2000 50  0001 C CNN
 F 3 "~" H 5600 2000 50  0001 C CNN
 	1    5600 2000
@@
 	6650 5550 6650 5600
 $Comp
-L Relay:G6S-2 K?
+L Relay:G6S-2 K1
 U 1 1 60844AEE
 P 7900 4400
-F 0 "K?" V 7133 4400 50  0000 C CNN
+F 0 "K1" V 7133 4400 50  0000 C CNN
 F 1 "G6S-2" V 7224 4400 50  0000 C CNN
-F 2 "" H 7900 4400 50  0001 L CNN
+F 2 "Relay_THT:Relay_DPDT_Omron_G6S-2" H 7900 4400 50  0001 L CNN
 F 3 "http://omronfs.omron.com/en_US/ecb/products/pdf/en-g6s.pdf" H 7900 4400 50  0001 C CNN
 	1    7900 4400
@@
 P 8350 3400
 AR Path="/60660B68/6084BE6E" Ref="#PWR?"  Part="1"
-AR Path="/607E0323/6084BE6E" Ref="#PWR?"  Part="1"
-F 0 "#PWR?" H 8350 3250 50  0001 C CNN
+AR Path="/607E0323/6084BE6E" Ref="#PWR098"  Part="1"
+F 0 "#PWR098" H 8350 3250 50  0001 C CNN
 F 1 "+24V" H 8365 3573 50  0000 C CNN
 F 2 "" H 8350 3400 50  0001 C CNN
@@
 	7500 4000 7600 4000
 $Comp
-L Diode:1N4148 D?
+L Diode:1N4148 D8
 U 1 1 608590BD
 P 7900 3500
-F 0 "D?" H 7900 3283 50  0000 C CNN
+F 0 "D8" H 7900 3283 50  0000 C CNN
 F 1 "1N4148" H 7900 3374 50  0000 C CNN
 F 2 "Diode_THT:D_DO-35_SOD27_P7.62mm_Horizontal" H 7900 3325 50  0001 C CNN
@@
 $EndComp
 $Comp
-L power:+5V #PWR?
+L power:+5V #PWR096
 U 1 1 60913ADA
 P 6800 1350
-F 0 "#PWR?" H 6800 1200 50  0001 C CNN
+F 0 "#PWR096" H 6800 1200 50  0001 C CNN
 F 1 "+5V" H 6815 1523 50  0000 C CNN
 F 2 "" H 6800 1350 50  0001 C CNN
@@
 	7350 1950 6800 1950
 $Comp
-L Connector:DB9_Female J?
+L Connector:DB9_Female J7
 U 1 1 60808F5E
 P 7650 1650
-F 0 "J?" H 7568 958 50  0000 C CNN
+F 0 "J7" H 7568 958 50  0000 C CNN
 F 1 "DB9_Female" H 7568 1049 50  0000 C CNN
-F 2 "" H 7650 1650 50  0001 C CNN
+F 2 "Connector_Dsub:DSUB-9_Female_Vertical_P2.77x2.84mm" H 7650 1650 50  0001 C CNN
 F 3 " ~" H 7650 1650 50  0001 C CNN
 	1    7650 1650
@@
 NoConn ~ 7350 1250
 $Comp
-L Device:Polyfuse F?
+L Device:Polyfuse F3
 U 1 1 60925B5A
 P 7150 1000
-F 0 "F?" V 6900 1000 50  0000 C CNN
+F 0 "F3" V 6900 1000 50  0000 C CNN
 F 1 "PFRA 050" V 7000 1000 50  0000 C CNN
 F 2 "Fuse:Fuse_BelFuse_0ZRE0005FF_L8.3mm_W3.8mm" H 6950 350 50  0001 C CNN
@@
 	7150 1350 7350 1350
 $Comp
-L Device:LED D?
+L Device:LED D7
 U 1 1 6092923F
 P 6950 4300
-F 0 "D?" V 6989 4182 50  0000 R CNN
+F 0 "D7" V 6989 4182 50  0000 R CNN
 F 1 "LED" V 6898 4182 50  0000 R CNN
-F 2 "" H 6950 4300 50  0001 C CNN
+F 2 "Diode_SMD:D_0603_1608Metric" H 6950 4300 50  0001 C CNN
 F 3 "~" H 6950 4300 50  0001 C CNN
 	1    6950 4300
@@
 	6650 4000 6950 4000
 $Comp
-L AR2ISS:R R?
+L AR2ISS:R R60
 U 1 1 6092E5F6
 P 6950 4650
-F 0 "R?" H 7020 4696 50  0000 L CNN
+F 0 "R60" H 7020 4696 50  0000 L CNN
 F 1 "3k" H 7020 4605 50  0000 L CNN
-F 2 "" V 6880 4650 50  0001 C CNN
+F 2 "Resistor_SMD:R_0603_1608Metric" V 6880 4650 50  0001 C CNN
 F 3 "~" H 6950 4650 50  0001 C CNN
 	1    6950 4650
