File: Rotor.sch (KiCad schematic (older format))
At the start: 33 parts

Commit message: first layout
Parts:
- removed C? (x4): 1n, symbol AR2ISS:C
- removed D? (x4): LED, symbol Device:LED
- removed L? (x4): 2.2u, symbol Device:L
- removed Q? (x4): AO3400A, Package_TO_SOT_SMD:SOT-23, symbol Transistor_FET:AO3400A
- removed R? (x4): 100k, symbol AR2ISS:R
- removed R? (x4): 220, symbol AR2ISS:R
- C29, C30: renamed from C?; footprint (none) -> Capacitor_SMD:C_0603_1608Metric
- L3, L4: renamed from L?; footprint (none) -> Inductor_SMD:L_0603_1608Metric
- R43, R44, R45, R46: renamed from R?; footprint (none) -> Resistor_SMD:R_0603_1608Metric
- gave numbers to parts that had none: 1
