File: PowerSupply.sch (KiCad schematic (older format))
At the start: 28 parts

Commit message: Ready for layout
Parts:
- removed C?: CP, symbol Device:CP
- added D? (x2): BZX84Cxx, Diode_SMD:D_SOT-23_ANK, symbol Diode:BZX84Cxx
- added F? (x2): PFRA 050, Fuse:Fuse_BelFuse_0ZRE0005FF_L8.3mm_W3.8mm, symbol Device:Polyfuse
- added L?: L, symbol Device:L
- R?: value .05 -> 0.1
- U?: value L7805 -> LME78_05-1.0; footprint (none) -> Package_TO_SOT_THT:TO-220-3_Vertical
Connections:
- net +12V: now also F?.2, F?.2; no longer C?.1, C?.1, C?.1, R?.2, U?.1 (IN), U?.4 (VN)
- net +3V3: no longer C?.1, U?.5 (VCC)
- net +5V: now also C?.1, U?.5 (VCC), L?.2; no longer C?.1, C?.1, C?.1, U?.3 (OUT)
- net ADC12V: now also D?.1 (K)
- net ADC24V: now also D?.1 (K)
- net GND: now also D?.2 (A), D?.2 (A)
- new net: C?.1, F?.1, R?.2, U?.4 (VN)
- new net: C?.1, C?.1, F?.1, U?.1 (IN)
- new net: C?.1, C?.1, C?.1, L?.1, U?.3 (OUT)
Other:
- moved on the sheet: C?, J?, Q?, R?, U?

Commit message: first layout
Parts:
- added J2: Conn_01x04, AR2ISS:250-204, symbol Connector_Generic:Conn_01x04
- C1, C10, C2, C6, C7: renamed from C?; value CP -> 22u; footprint (none) -> Capacitor_THT:CP_Radial_D6.3mm_P2.50mm
- C11, C12, C13, C3, C4, C5, C8, C9: renamed from C?; footprint (none) -> Capacitor_SMD:C_0603_1608Metric
- J1: renamed from J?; footprint (none) -> stmbl:RM3.5_1x2
- L1: renamed from L?; footprint (none) -> Inductor_SMD:L_0603_1608Metric
- Q2: renamed from Q?; footprint (none) -> Package_SO:SO-8_5.3x6.2mm_P1.27mm
- R10, R11, R4, R5, R6, R7, R9: renamed from R?; footprint (none) -> Resistor_SMD:R_0603_1608Metric
- R8: renamed from R?; footprint (none) -> Resistor_SMD:R_1206_3216Metric_Pad1.30x1.75mm_HandSolder
- U6: renamed from U?; footprint (none) -> Package_TO_SOT_SMD:SOT-223
- gave numbers to parts that had none: 7
Connections:
- net +12V: now also J2.2 (Pin_2)
- net +24V: now also J2.1 (Pin_1)
- net GND: now also J2.3 (Pin_3), J2.4 (Pin_4)

Commit message: ready for ordering
Parts:
- Q2: footprint Package_SO:SO-8_5.3x6.2mm_P1.27mm -> Package_TO_SOT_SMD:SOT-363_SC-70-6_Handsoldering; symbol Device:Q_PMOS_DGS -> Transistor_FET:Si1442DH
Connections:
- net at C12.2, R8.1, R9.1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: now also Q2.4 (S); no longer Q2.3 (S)
- net at J1.1 (Pin_1), Q2.1 (D): now also Q2.2 (D), Q2.5 (D), Q2.6 (D)
- net at R11.1, R9.2: now also Q2.3 (G); no longer Q2.2 (G)
Changed lines of the file:
@@
 $EndComp
 $Comp
-L Device:Q_PMOS_DGS Q2
+L Transistor_FET:Si1442DH Q2
 U 1 1 606B052C
 P 5350 1750
 F 0 "Q2" V 5692 1750 50  0000 C CNN
 F 1 "APM4953KC" V 5601 1750 50  0000 C CNN
-F 2 "Package_SO:SO-8_5.3x6.2mm_P1.27mm" H 5550 1850 50  0001 C CNN
+F 2 "Package_TO_SOT_SMD:SOT-363_SC-70-6_Handsoldering" H 5550 1850 50  0001 C CNN
 F 3 "~" H 5350 1750 50  0001 C CNN
 	1    5350 1750
