File: filter.sch (KiCad schematic (older format))
At the start: 13 parts, among them J13 Conn_01x02

Commit message: ready for ordering
Parts:
- D12: value PESD2CAN -> PSM712-LF-T7
Changed lines of the file:
@@
 $Descr A4 11693 8268
 encoding utf-8
-Sheet 19 21
+Sheet 21 21
 Title ""
 Date ""
@@
 AR Path="/6072829D/60797D2F/60999526/609A19E2" Ref="L15"  Part="1"
 AR Path="/6072829D/607938CE/60999526/609A19E2" Ref="L19"  Part="1"
-F 0 "L19" V 5540 3000 50  0000 C CNN
+F 0 "L23" V 5540 3000 50  0000 C CNN
 F 1 "74279266" V 5449 3000 50  0000 C CNN
 F 2 "Inductor_SMD:L_0603_1608Metric" H 5350 3000 50  0001 C CNN
@@
 AR Path="/6072829D/60797D2F/60999526/609A19E8" Ref="R72"  Part="1"
 AR Path="/6072829D/607938CE/60999526/609A19E8" Ref="R79"  Part="1"
-F 0 "R79" H 6770 3346 50  0000 L CNN
+F 0 "R86" H 6770 3346 50  0000 L CNN
 F 1 "220" H 6770 3255 50  0000 L CNN
 F 2 "Resistor_SMD:R_0603_1608Metric" V 6630 3300 50  0001 C CNN
@@
 AR Path="/6072829D/60797D2F/60999526/609A19EE" Ref="C44"  Part="1"
 AR Path="/6072829D/607938CE/60999526/609A19EE" Ref="C49"  Part="1"
-F 0 "C49" H 6815 3746 50  0000 L CNN
+F 0 "C54" H 6815 3746 50  0000 L CNN
 F 1 "1n" H 6815 3655 50  0000 L CNN
 F 2 "Capacitor_SMD:C_0603_1608Metric" H 6738 3550 50  0001 C CNN
@@
 AR Path="/6072829D/60797D2F/60999526/609A19F4" Ref="C42"  Part="1"
 AR Path="/6072829D/607938CE/60999526/609A19F4" Ref="C47"  Part="1"
-F 0 "C47" H 6315 3346 50  0000 L CNN
+F 0 "C52" H 6315 3346 50  0000 L CNN
 F 1 "470p" H 6315 3255 50  0000 L CNN
 F 2 "Capacitor_SMD:C_0603_1608Metric" H 6238 3150 50  0001 C CNN
@@
 AR Path="/6072829D/60797D2F/60999526/609A19FA" Ref="L17"  Part="1"
 AR Path="/6072829D/607938CE/60999526/609A19FA" Ref="L21"  Part="1"
-F 0 "L21" V 7740 3000 50  0000 C CNN
+F 0 "L25" V 7740 3000 50  0000 C CNN
 F 1 "10u" V 7649 3000 50  0000 C CNN
 F 2 "Inductor_SMD:L_0603_1608Metric" H 7550 3000 50  0001 C CNN
@@
 AR Path="/6072829D/60797D2F/60999526/609A1A04" Ref="#PWR0111"  Part="1"
 AR Path="/6072829D/607938CE/60999526/609A1A04" Ref="#PWR0117"  Part="1"
-F 0 "#PWR0117" H 6700 3750 50  0001 C CNN
+F 0 "#PWR0123" H 6700 3750 50  0001 C CNN
 F 1 "GND" H 6705 3827 50  0000 C CNN
 F 2 "" H 6700 4000 50  0001 C CNN
@@
 AR Path="/6072829D/60797D2F/60999526/609A1A0B" Ref="#PWR0112"  Part="1"
 AR Path="/6072829D/607938CE/60999526/609A1A0B" Ref="#PWR0118"  Part="1"
-F 0 "#PWR0118" H 6200 3750 50  0001 C CNN
+F 0 "#PWR0124" H 6200 3750 50  0001 C CNN
 F 1 "GND" H 6205 3827 50  0000 C CNN
 F 2 "" H 6200 4000 50  0001 C CNN
@@
 AR Path="/6072829D/60797D2F/60999526/609A1A16" Ref="L14"  Part="1"
 AR Path="/6072829D/607938CE/60999526/609A1A16" Ref="L18"  Part="1"
-F 0 "L18" V 5540 1500 50  0000 C CNN
+F 0 "L22" V 5540 1500 50  0000 C CNN
 F 1 "74279266" V 5449 1500 50  0000 C CNN
 F 2 "Inductor_SMD:L_0603_1608Metric" H 5350 1500 50  0001 C CNN
@@
 AR Path="/6072829D/60797D2F/60999526/609A1A1C" Ref="R71"  Part="1"
 AR Path="/6072829D/607938CE/60999526/609A1A1C" Ref="R78"  Part="1"
-F 0 "R78" H 6770 1846 50  0000 L CNN
+F 0 "R85" H 6770 1846 50  0000 L CNN
 F 1 "220" H 6770 1755 50  0000 L CNN
 F 2 "Resistor_SMD:R_0603_1608Metric" V 6630 1800 50  0001 C CNN
@@
 AR Path="/6072829D/60797D2F/60999526/609A1A22" Ref="C43"  Part="1"
 AR Path="/6072829D/607938CE/60999526/609A1A22" Ref="C48"  Part="1"
-F 0 "C48" H 6815 2246 50  0000 L CNN
+F 0 "C53" H 6815 2246 50  0000 L CNN
 F 1 "1n" H 6815 2155 50  0000 L CNN
 F 2 "Capacitor_SMD:C_0603_1608Metric" H 6738 2050 50  0001 C CNN
@@
 AR Path="/6072829D/60797D2F/60999526/609A1A28" Ref="C41"  Part="1"
 AR Path="/6072829D/607938CE/60999526/609A1A28" Ref="C46"  Part="1"
-F 0 "C46" H 6315 1846 50  0000 L CNN
+F 0 "C51" H 6315 1846 50  0000 L CNN
 F 1 "470p" H 6315 1755 50  0000 L CNN
 F 2 "Capacitor_SMD:C_0603_1608Metric" H 6238 1650 50  0001 C CNN
@@
 AR Path="/6072829D/60797D2F/60999526/609A1A2E" Ref="L16"  Part="1"
 AR Path="/6072829D/607938CE/60999526/609A1A2E" Ref="L20"  Part="1"
-F 0 "L20" V 7740 1500 50  0000 C CNN
+F 0 "L24" V 7740 1500 50  0000 C CNN
 F 1 "10u" V 7649 1500 50  0000 C CNN
 F 2 "Inductor_SMD:L_0603_1608Metric" H 7550 1500 50  0001 C CNN
@@
 AR Path="/6072829D/60797D2F/60999526/609A1A38" Ref="#PWR0113"  Part="1"
 AR Path="/6072829D/607938CE/60999526/609A1A38" Ref="#PWR0119"  Part="1"
-F 0 "#PWR0119" H 6700 2250 50  0001 C CNN
+F 0 "#PWR0125" H 6700 2250 50  0001 C CNN
 F 1 "GND" H 6705 2327 50  0000 C CNN
 F 2 "" H 6700 2500 50  0001 C CNN
@@
 AR Path="/6072829D/60797D2F/60999526/609A1A3F" Ref="#PWR0114"  Part="1"
 AR Path="/6072829D/607938CE/60999526/609A1A3F" Ref="#PWR0120"  Part="1"
-F 0 "#PWR0120" H 6200 2250 50  0001 C CNN
+F 0 "#PWR0126" H 6200 2250 50  0001 C CNN
 F 1 "GND" H 6205 2327 50  0000 C CNN
 F 2 "" H 6200 2500 50  0001 C CNN
@@
 AR Path="/6072829D/60797D2F/60999526/609A1A59" Ref="J11"  Part="1"
 AR Path="/6072829D/607938CE/60999526/609A1A59" Ref="J12"  Part="1"
-F 0 "J12" H 4318 2367 50  0000 C CNN
+F 0 "J13" H 4318 2367 50  0000 C CNN
 F 1 "Conn_01x02" H 4318 2276 50  0000 C CNN
 F 2 "Connector_PinHeader_2.54mm:PinHeader_1x02_P2.54mm_Vertical" H 4400 2150 50  0001 C CNN
@@
 AR Path="/6072829D/60797D2F/60999526/609A1A5F" Ref="R66"  Part="1"
 AR Path="/6072829D/607938CE/60999526/609A1A5F" Ref="R73"  Part="1"
-F 0 "R73" H 4270 2696 50  0000 L CNN
+F 0 "R80" H 4270 2696 50  0000 L CNN
 F 1 "120" H 4270 2605 50  0000 L CNN
 F 2 "Resistor_SMD:R_0603_1608Metric" V 4130 2650 50  0001 C CNN
@@
 AR Path="/6072829D/60797D2F/60999526/609A1A67" Ref="#PWR0115"  Part="1"
 AR Path="/6072829D/607938CE/60999526/609A1A67" Ref="#PWR0121"  Part="1"
-F 0 "#PWR0121" H 3450 2150 50  0001 C CNN
+F 0 "#PWR0129" H 3450 2150 50  0001 C CNN
 F 1 "GND" H 3455 2227 50  0000 C CNN
 F 2 "" H 3450 2400 50  0001 C CNN
@@
 AR Path="/6072829D/60797D2F/60999526/609A1A6F" Ref="D10"  Part="1"
 AR Path="/6072829D/607938CE/60999526/609A1A6F" Ref="D11"  Part="1"
-F 0 "D11" V 3154 2330 50  0000 L CNN
-F 1 "PESD2CAN" V 3245 2330 50  0000 L CNN
+F 0 "D12" V 3154 2330 50  0000 L CNN
+F 1 "PSM712-LF-T7" V 3245 2330 50  0000 L CNN
 F 2 "Package_TO_SOT_SMD:SOT-23_Handsoldering" H 3050 2250 50  0001 C CNN
 F 3 "~" H 3050 2250 50  0001 C CNN
